File: PCB-Legos/Antenna tester/HGS_antenna_tester.kicad_sch (KiCad schematic)
At the start: 5 parts

Commit message: stictching and typo fixes
Parts:
- J1: value (none) -> Conn_Coaxial; footprint (none) -> Connector_Coaxial:SMA_Amphenol_132134-10_Vertical
- J2: value (none) -> Conn_01x01; footprint (none) -> Connector_Wire:SolderWire-0.5sqmm_1x01_D0.9mm_OD2.1mm
- R1, R3: value (none) -> DNP; footprint (none) -> Resistor_SMD:R_0402_1005Metric_Pad0.72x0.64mm_HandSolder
- R2: value (none) -> 0; footprint (none) -> Resistor_SMD:R_0402_1005Metric_Pad0.72x0.64mm_HandSolder
Other:
- note added: "Antenna wire connection 20AWG (0.5mm^2) mag wire"
- note added: "Resistors are place holders can be: - Resistors - Capacitors - Inductors"
- note removed: "Antenna wire connection 20AWG mag wire"
- note removed: "Resistors are place holders can be: - Restors - Capacitors - Inductors"
Changed lines of the file:
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@@
     (stroke (width 0) (type default) (color 0 0 0 0))
   )
-  (text "Antenna wire connection\n20AWG mag wire\n\n" (at 161.29 92.71 0)
+  (text "Antenna wire connection\n20AWG (0.5mm^2) mag wire\n\n"
+    (at 161.29 92.71 0)
     (effects (font (size 1.27 1.27)) (justify left bottom))
   )
@@
     (effects (font (size 1.27 1.27)) (justify left bottom))
   )
-  (text "Resistors are place holders\ncan be:\n- Restors\n- Capacitors\n- Inductors"
+  (text "Resistors are place holders\ncan be:\n- Resistors\n- Capacitors\n- Inductors"
     (at 125.73 129.54 0)
     (effects (font (size 1.27 1.27)) (justify left bottom))
@@
       (effects (font (size 1.27 1.27)) (justify left))
     )
-    (property "Value" "" (id 1) (at 151.13 106.6799 0)
+    (property "Value" "DNP" (id 1) (at 151.13 106.6799 0)
       (effects (font (size 1.27 1.27)) (justify left))
     )
-    (property "Footprint" "" (id 2) (at 148.59 105.41 0)
+    (property "Footprint" "Resistor_SMD:R_0402_1005Metric_Pad0.72x0.64mm_HandSolder" (id 2) (at 148.59 105.41 0)
       (effects (font (size 1.27 1.27)) hide)
     )
@@
     (in_bom yes) (on_board yes) (fields_autoplaced)
     (property "Reference" "J1" (id 0) (at 110.8074 92.71 0))
-    (property "Value" "" (id 1) (at 110.8074 95.25 0))
-    (property "Footprint" "" (id 2) (at 110.49 100.33 0)
+    (property "Value" "Conn_Coaxial" (id 1) (at 110.8074 95.25 0))
+    (property "Footprint" "Connector_Coaxial:SMA_Amphenol_132134-10_Vertical" (id 2) (at 110.49 100.33 0)
       (effects (font (size 1.27 1.27)) hide)
     )
@@
       (effects (font (size 1.27 1.27)) (justify left))
     )
-    (property "Value" "" (id 1) (at 173.99 101.5999 0)
+    (property "Value" "Conn_01x01" (id 1) (at 173.99 101.5999 0)
       (effects (font (size 1.27 1.27)) (justify left))
     )
-    (property "Footprint" "" (id 2) (at 171.45 100.33 0)
+    (property "Footprint" "Connector_Wire:SolderWire-0.5sqmm_1x01_D0.9mm_OD2.1mm" (id 2) (at 171.45 100.33 0)
       (effects (font (size 1.27 1.27)) hide)
     )
@@
       (effects (font (size 1.27 1.27)) (justify left))
     )
-    (property "Value" "" (id 1) (at 132.08 106.6799 0)
+    (property "Value" "DNP" (id 1) (at 132.08 106.6799 0)
       (effects (font (size 1.27 1.27)) (justify left))
     )
-    (property "Footprint" "" (id 2) (at 129.54 105.41 0)
+    (property "Footprint" "Resistor_SMD:R_0402_1005Metric_Pad0.72x0.64mm_HandSolder" (id 2) (at 129.54 105.41 0)
       (effects (font (size 1.27 1.27)) hide)
     )
@@
       (effects (font (size 1.27 1.27)) hide)
     )
-    (property "Value" "" (id 1) (at 129.54 115.57 0))
+    (property "Value" "GND" (id 1) (at 129.54 115.57 0))
     (property "Footprint" "" (id 2) (at 129.54 110.49 0)
       (effects (font (size 1.27 1.27)) hide)
@@
     (in_bom yes) (on_board yes) (fields_autoplaced)
     (property "Reference" "R2" (id 0) (at 139.7 93.98 90))
-    (property "Value" "" (id 1) (at 139.7 96.52 90))
-    (property "Footprint" "" (id 2) (at 139.7 100.33 0)
+    (property "Value" "0" (id 1) (at 139.7 96.52 90))
+    (property "Footprint" "Resistor_SMD:R_0402_1005Metric_Pad0.72x0.64mm_HandSolder" (id 2) (at 139.7 100.33 0)
       (effects (font (size 1.27 1.27)) hide)
     )
