File: PCB-Legos/LNA/LNA.kicad_pcb (KiCad board)
At the start: 4 copper layers, 50.8 x 24.6 mm, 42 parts, among them J1 Conn_Coaxial, J2 Conn_Coaxial, J3 Conn_Coaxial, J4 474-PRT-00587, U1 LP2985XX-N, U2 LNA-TP3M9037, U3 QPQ1907, U4 LP2985XX-N, U5 LNA-TP3M9037, U6 QPQ1907

Commit message: LNA Test Board
Reviewed work done during capstone. Everything seems ready to build and test.
Routing:
- net Net-(C3-Pad2): track 11.3 -> 15.3 mm
Changed lines of the file:
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@@
   (segment (start 142.062037 76.950628) (end 142.1512 77.039791) (width 0.25) (layer "F.Cu") (net 30))
   (segment (start 138.284242 76.118749) (end 138.6332 75.769791) (width 0.25) (layer "F.Cu") (net 30))
+  (segment (start 138.468 70.5104) (end 140.8556 70.5104) (width 0.25) (layer "F.Cu") (net 30))
   (segment (start 138.468 71.92) (end 139.192 72.644) (width 0.25) (layer "F.Cu") (net 30))
   (segment (start 138.6332 75.769791) (end 139.269791 75.769791) (width 0.25) (layer "F.Cu") (net 30))
+  (segment (start 140.8556 70.5104) (end 141.960142 69.405858) (width 0.25) (layer "F.Cu") (net 30))
   (segment (start 138.468 70.5104) (end 138.468 71.92) (width 0.25) (layer "F.Cu") (net 30))
   (segment (start 142.07474 77.116251) (end 142.1512 77.039791) (width 0.25) (layer "F.Cu") (net 30))

Commit message: 50 Ohm microstrip
Test boards with a through, impedance matching network and 50ohm load test
Parts:
- moved C10 10.9 mm to (148.8, 67.9)
- turned C3 to 180 degrees
Routing:
- net Net-(C10-Pad2): track 10.4 -> 14.2 mm
- net Net-(C3-Pad2): track 15.3 -> 12.0 mm
- net GND: track 8.71 -> 8.42 mm, vias 102 -> 106
Other:
- board size 50.8 x 24.6 mm -> 51.1 x 24.8 mm
- board text added: "LNA Test Board v2"
- board text removed: "KK7AQM teehee"
- board text removed: "LNA Test Board v1"
