File: PCB-Legos/Antenna tester/50_ohm_microstrip_experiment/50_ohm_microstrip_experiment.kicad_pcb (KiCad board)
At the start: 4 copper layers, 45.7 x 66.5 mm, 10 parts, among them J1 Conn_Coaxial, J3 Conn_Coaxial, J4 Conn_Coaxial, J5 Conn_Coaxial

Commit message: Added designators and fixed soldermask removal
Added designators and fixed soldermask removal
Also added board title
Parts:
- R5: value 150 -> ~150 ohm
- R6: renamed from R5; value 150 -> 50 ohm
- renumbered J3 to J4, J4 to J6
Other:
- board text added: "50 ohm sanity check"
- board text added: "Impedance Matching @ 2.42GHz V2"
- board text added: "L Match"
- board text added: "Open stub"
- board text added: "Through"
Changed lines of the file:
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@@
     (property "Sheetname" "")
     (attr smd)
-    (fp_text reference "J3" (at 1.1176 -5.6896 -90 unlocked) (layer "F.SilkS") hide
+    (fp_text reference "J4" (at -4.5466 3.8608 -90 unlocked) (layer "F.SilkS")
       (effects (font (size 1 1) (thickness 0.15)))
     )
@@
       (effects (font (size 0.17 0.17) (thickness 0.03)))
     )
-    (fp_text value "150" (at -0.7 1.25) (layer "F.Fab")
+    (fp_text value "~150 ohm" (at -4.699 -2.667) (layer "F.SilkS")
       (effects (font (size 0.68 0.68) (thickness 0.12)) (justify right bottom))
     )
@@
       (effects (font (size 0.17 0.17) (thickness 0.03)))
     )
-    (fp_text value "7nH" (at 1.27 -0.3556 90) (layer "F.Fab")
+    (fp_text value "7nH" (at 2.0574 -0.3302 90) (layer "F.SilkS")
       (effects (font (size 0.68 0.68) (thickness 0.12)) (justify right bottom))
     )
@@
     (property "Sheetfile" "50_ohm_microstrip_experiment.kicad_sch")
     (property "Sheetname" "")
-    (fp_text reference "R5" (at 0 0) (layer "F.Mask")
+    (fp_text reference "R6" (at 0 0) (layer "F.Mask") hide
       (effects (font (size 0.17 0.17) (thickness 0.03)))
     )
-    (fp_text value "150" (at -0.7 1.25) (layer "F.Fab")
+    (fp_text value "50 ohm" (at -0.9906 2.7178) (layer "F.SilkS")
       (effects (font (size 0.68 0.68) (thickness 0.12)) (justify left bottom))
     )
@@
     (property "Sheetname" "")
     (attr smd)
-    (fp_text reference "J4" (at 0 0.1651 -90 unlocked) (layer "F.SilkS") hide
+    (fp_text reference "J6" (at -4.4196 3.8323 -90 unlocked) (layer "F.SilkS")
       (effects (font (size 1 1) (thickness 0.15)))
     )
@@
     (property "Sheetname" "")
     (attr smd)
-    (fp_text reference "J1" (at 3.429 -0.0889 90 unlocked) (layer "F.SilkS") hide
+    (fp_text reference "J1" (at 4.445 3.81 90 unlocked) (layer "F.SilkS")
       (effects (font (size 1 1) (thickness 0.15)))
     )
@@
     (property "Sheetname" "")
     (attr smd)
-    (fp_text reference "J3" (at 1.1176 -5.6896 90 unlocked) (layer "F.SilkS")
+    (fp_text reference "J3" (at 4.318 3.7592 90 unlocked) (layer "F.SilkS")
       (effects (font (size 1 1) (thickness 0.15)))
     )
@@
     (property "Sheetname" "")
     (attr smd)
-    (fp_text reference "J5" (at 0 0.1651 90 unlocked) (layer "F.SilkS") hide
+    (fp_text reference "J5" (at 4.4196 3.8323 90 unlocked) (layer "F.SilkS")
       (effects (font (size 1 1) (thickness 0.15)))
     )
@@
       (effects (font (size 0.17 0.17) (thickness 0.03)))
     )
-    (fp_text value ".9pF" (at -1.4478 2.413) (layer "F.Fab")
+    (fp_text value ".9pF" (at -1.9304 2.7178) (layer "F.SilkS")
       (effects (font (size 0.68 0.68) (thickness 0.12)) (justify left bottom))
     )
@@
   )
   (gr_rect (start 131.064 30.226) (end 176.784 96.774) (layer "Edge.Cuts") (width 0.2) (fill none))
+  (gr_text "50 ohm sanity check" (at 165.3032 61.6966) (layer "F.SilkS")
+    (effects (font (size 0.7 0.7) (thickness 0.175)))
+  )
+  (gr_text "L Match" (at 141.0716 61.3664) (layer "F.SilkS")
+    (effects (font (size 0.7 0.7) (thickness 0.175)))
+  )
+  (gr_text "Through" (at 140.6398 35.9156) (layer "F.SilkS")
+    (effects (font (size 0.7 0.7) (thickness 0.175)))
+  )
+  (gr_text "Impedance Matching @ 2.42GHz V2" (at 165.5826 93.8784) (layer "F.SilkS")
+    (effects (font (size 1 0.8) (thickness 0.2)))
+  )
+  (gr_text "Open stub" (at 141.2494 81.8642) (layer "F.SilkS")
+    (effects (font (size 0.7 0.7) (thickness 0.175)))
+  )
   (segment (start 165.989 64.2112) (end 165.9636 64.1858) (width 0.25) (layer "F.Cu") (net 1))
   (segment (start 142.0042 64.1096) (end 142.8242 64.1096) (width 0.38) (layer "F.Cu") (net 1))
@@
     (polygon
       (pts
-        (xy 162.2298 88.7476)
+        (xy 162.8902 88.7476)
         (xy 129.54 88.7476)
         (xy 129.54 83.6168)
-        (xy 162.2298 83.6168)
+        (xy 162.8902 83.6168)
       )
     )
@@
     (connect_pads (clearance 0))
     (min_thickness 0.254) (filled_areas_thickness no)
-    (fill yes (thermal_gap 0.508) (thermal_bridge_width 0.508))
-    (polygon
-      (pts
-        (xy 142.2146 64.3128)
-        (xy 136.2964 64.3128)
-        (xy 136.2964 63.9064)
-        (xy 142.2146 63.9064)
+    (fill (thermal_gap 0.508) (thermal_bridge_width 0.508))
+    (polygon
+      (pts
+        (xy 142.2654 65.405)
+        (xy 131.318 65.405)
+        (xy 131.318 62.738)
+        (xy 142.2654 62.738)
       )
     )
@@
     (connect_pads (clearance 0))
     (min_thickness 0.254) (filled_areas_thickness no)
-    (fill yes (thermal_gap 0.508) (thermal_bridge_width 0.508))
-    (polygon
-      (pts
-        (xy 172.1104 39.4208)
-        (xy 135.6868 39.4208)
-        (xy 135.6868 39.0144)
-        (xy 172.1104 39.0144)
+    (fill (thermal_gap 0.508) (thermal_bridge_width 0.508))
+    (polygon
+      (pts
+        (xy 176.5808 40.4876)
+        (xy 131.3942 40.4876)
+        (xy 131.3942 37.8714)
+        (xy 176.5808 37.8714)
       )
     )
@@
     (connect_pads (clearance 0))
     (min_thickness 0.254) (filled_areas_thickness no)
-    (fill yes (thermal_gap 0.508) (thermal_bridge_width 0.508))
-    (polygon
-      (pts
-        (xy 147.447 92.075)
-        (xy 146.685 92.075)
-        (xy 146.685 86.5632)
-        (xy 147.447 86.5632)
+    (fill (thermal_gap 0.508) (thermal_bridge_width 0.508))
+    (polygon
+      (pts
+        (xy 149.6314 93.3704)
+        (xy 144.4752 93.3704)
+        (xy 144.4752 86.5632)
+        (xy 149.6314 86.5632)
       )
     )
@@
     (connect_pads (clearance 0))
     (min_thickness 0.254) (filled_areas_thickness no)
-    (fill yes (thermal_gap 0.508) (thermal_bridge_width 0.508))
-    (polygon
-      (pts
-        (xy 162.0012 86.5632)
-        (xy 130.9624 86.5632)
-        (xy 130.9624 85.8012)
-        (xy 162.0012 85.8012)
+    (fill (thermal_gap 0.508) (thermal_bridge_width 0.508))
+    (polygon
+      (pts
+        (xy 162.8902 88.7476)
+        (xy 130.9624 88.7476)
+        (xy 130.9624 83.6168)
+        (xy 162.8902 83.6168)
       )
     )
@@
     (connect_pads (clearance 0))
     (min_thickness 0.254) (filled_areas_thickness no)
-    (fill yes (thermal_gap 0.508) (thermal_bridge_width 0.508))
-    (polygon
-      (pts
-        (xy 165.8112 64.008)
-        (xy 176.657 64.008)
-        (xy 176.657 64.4144)
-        (xy 165.8112 64.4144)
-      )
-    )
+    (fill (thermal_gap 0.508) (thermal_bridge_width 0.508))
+    (polygon
+      (pts
+        (xy 165.6842 62.9158)
+        (xy 176.657 62.9158)
+        (xy 176.657 65.5828)
+        (xy 165.6842 65.5828)
+      )
+    )
