File: pcba/KiCad/HGS_Reflector.kicad_sch (KiCad schematic)
At the start: 57 parts, among them J1 U.FL, J2 USB_MINI-B_SMT, J3 SM06B-SRSS-TB(LF)(SN), J5 132134-10, J6 132134-10, J7 USB_HOST_W{slash}CHASSIS_GND, T1 QWT2.4222, U1 LP2985XX-N, U2 LP2985XX-N, U3 NCS3-272+, U4 QPQ1907, U5 QPQ1907, U6 LNA-TP3M9037, U7 LNA-TP3M9037

Commit message: replaced some eagle import symbols with kicad symbols
Parts:
- removed J2: USB_MINI-B_SMT, USB-MINIB, symbol HGS_Reflector-eagle-import:USB_MINI-B_SMT
- removed TP2: TEST-POINT-LARGE-SQUARE, 1X01, symbol HGS_Reflector-eagle-import:TEST-POINT-LARGE-SQUARE
- removed U1, U2: LP2985XX-N, SOT-23, symbol HGS_Reflector-eagle-import:LP2985XX-N
- removed U5: QPQ1907, QPQ1907, symbol HGS_Reflector-eagle-import:QPQ1907
- removed U6, U7: LNA-TP3M9037, TP3M9037, symbol HGS_Reflector-eagle-import:LNA-TP3M9037
- added P1: USB_C_Plug_USB2.0, symbol Connector:USB_C_Plug_USB2.0
- added TP1: Test-Point, oresat-misc:TestPoint-0.75mm-th, symbol oresat-misc:Test-Point-0.75mm-th
- added U1, U5: LP2985-N, Package_TO_SOT_SMD:SOT-23-5, symbol oresat-ics:LP2985-N
- added U2, U7: TQP3M9037, SON50P200X200X95-9N-D, symbol oresat-ics:TQP3M9037_1
- added U8: ~, Bidirectional_Amp:FIL_B39162B9417K610, symbol oresat-ics:QPQ1907
- C1, C11, C12, C2, C21, C9: symbol HGS_Reflector-eagle-import:C-EU0603-C-NOSILK -> Device:C_Small
- C10, C13, C15, C16, C17, C20, C5, C7, C8: symbol HGS_Reflector-eagle-import:C-EU0603-B-NOSILK -> Device:C_Small
- C14, C18, C19, C3, C4, C6: symbol HGS_Reflector-eagle-import:C-EU0402-C-NOSILK -> Device:C_Small
- E1, E2, E3, E4, E5: symbol HGS_Reflector-eagle-import:L-BEAD-0603-B -> Device:FerriteBead_Small
- J7: symbol HGS_Reflector-eagle-import:USB_HOST_W/CHASSIS_GND -> HGS_Reflector-eagle-import:USB_HOST_W/CHASSIS_GND
- L1, L2: value 10 nH -> 10n
- L3, L4: value 8 nH -> 8n
- R1, R2, R3, R5, R6, R7, R9: symbol HGS_Reflector-eagle-import:R-US_0603-B-NOSILK -> Device:R_Small_US
- R4: symbol HGS_Reflector-eagle-import:R-US_0402-C-NOSILK -> Device:R_Small_US
- U4: footprint QPQ1907 -> oresat-ics:QPQ1907SR; symbol HGS_Reflector-eagle-import:QPQ1907 -> oresat-ics:QPQ1907
Connections:
- net GND: now also U4.2 (GND), U4.3 (GND), U4.5 (GND), P1.A1 (GND), P1.A12 (GND), P1.B1 (GND), P1.B12 (GND), U1.2 (GND), U2.6 (SHUT_DOWN), U2.9 (GND), U5.2 (GND), U7.6 (SHUT_DOWN), U7.9 (GND), U8.2 (GND), U8.3 (GND), U8.5 (GND); no longer U4.GND, U4.GND2 (GND), U4.GND3 (GND)
- net at C8.1, R3.1: now also U1.5 (VOUT)
- net at C15.1: now also U5.4 (BYPASS)
- net at C16.1, R5.1: now also U5.5 (VOUT)
- net at C4.2: now also U8.1 (IN)
- net at J1.FEED (SIGNAL): now also U8.4 (OUT)
- net at C4.1, L1.1: now also U7.7 (RF_OUT)
- net at C14.1, L2.1: now also U2.7 (RF_OUT)
- net at C14.2: now also U4.1 (IN); no longer U4.INPUT (RF_IN)
- net at J7.1 (VBUS): now also TP1.1
- net at C3.1: now also U4.4 (OUT); no longer U4.OUTPUT (RF-OUT)
- net at C3.2: now also U7.2 (RF_IN)
- net at C9.2: now also P1.S1 (SHIELD)
- net at C7.1: now also U1.4 (BYPASS)
- net at E4.1: now also P1.A4 (VBUS), P1.A9 (VBUS), P1.B4 (VBUS), P1.B9 (VBUS)
- net at C6.2: now also U2.2 (RF_IN)
- net VUSB renamed VBUS
- net VBUS: now also U1.1 (VIN), U1.3 (EN), U5.1 (VIN), U5.3 (EN)
- no-connect marks 0 -> 4

Commit message: deleted temp files
Parts:
- U8: value ~ -> B39162B9417K610
Other:
- note added: "NCS3-72+?"
- note added: "Power"
- note added: "Qualcomm Atheros AR9721?"
- note added: "RF Front-end"
- note added: "U8 is obsolete. Suggested replacement is B3916B9417K810"
- moved on the sheet: C1, C10, C11, C12, C13, C14, C15, C16, C18, C19, C2, C3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

Commit message: cleanup of kicad files
Other:
- title: (none) -> OreSat Live Handheld Ground Station
Changed lines of the file:
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@@
 	(generator "eeschema")
 	(generator_version "8.0")
-	(paper "USLedger")
+	(paper "B")
+	(title_block
+		(title "OreSat Live Handheld Ground Station")
+		(date "2024-09-10")
+		(rev "2")
+	)
 	(junction
 		(at 172.72 184.15)

Commit message: fixed reference designators, fixed symbol/footprint pads and pins, added impedance matching at helical
Parts:
- removed J6: 132134-10, 132134-10, symbol HGS_Reflector-eagle-import:132134-10
- removed LED1, LED2: GREEN, LED-0603, symbol HGS_Reflector-eagle-import:LED-GREEN0603
- removed R4: 150, .0402-C-NOSILK, symbol Device:R_Small_US
- removed T1: QWT2.4222, QWT_2.422G-V2, symbol HGS_Reflector-eagle-import:QWT2.4222
- removed U3: NCS3-272+, GE0805C-1, symbol HGS_Reflector-eagle-import:NCS3-272+
- added C22: 1.0 pF, oresat-passives:0402-C-NOSILK, symbol Device:C_Small
- added D1, D2: Green, LED_SMD:LED_0603_1608Metric_Pad1.05x0.95mm_HandSolder, symbol Device:LED_Small
- added L5: 4.3 nH, oresat-passives:0402-C-NOSILK, symbol Device:L
- C1, C11, C12, C2, C21, C9: footprint .0603-C-NOSILK -> oresat-passives:0603-C-NOSILK
- C10, C13, C15, C16, C17, C20, C5, C7, C8, R1, R2, R3, R5, R6, R7, R9: footprint .0603-B-NOSILK -> oresat-passives:0603-B-NOSILK
- C14, C18, C3, C4, C6: footprint .0402-C-NOSILK -> oresat-passives:0402-C-NOSILK
- C19: value 100 pF -> 0.9 pF; footprint .0402-C-NOSILK -> oresat-passives:0402-C-NOSILK; MPN (none) -> 04025J0R9PBSTR
- E1, E2, E3, E4, E5: footprint .0603-B -> oresat-passives:0603-B-NOSILK
- J1: footprint U.FL -> oresat-connectors:U.FL; symbol HGS_Reflector-eagle-import:U.FL -> oresat-connectors:U.FL
- J2: renamed from P1; footprint (none) -> oresat-connectors:USB-MINIB
- J3: footprint CONN_SM06B-SRSS-TB_JST -> oresat-connectors:CONN_SM06B-SRSS-TB_JST; symbol HGS_Reflector-eagle-import:SM06B-SRSS-TB(LF)(SN) -> oresat-connectors:SM06B-SRSS-TB(LF)(SN); Distributor (none) -> DigiKey; MPN (none) -> SM06B-SRSS-TB(LF)(SN)
- J5: footprint 132134-10 -> oresat-connectors:U.FL; symbol HGS_Reflector-eagle-import:132134-10 -> oresat-connectors:U.FL
- J7: footprint GHI2_USB_HOST_HORIZONTAL_W_CHASSIS_GND -> oresat-misc:GHI2_USB_HOST_HORIZONTAL_W_CHASSIS_GND; symbol HGS_Reflector-eagle-import:USB_HOST_W/CHASSIS_GND -> oresat-misc:USB_HOST_W/CHASSIS_GND
- L1, L2, L3, L4: footprint L3216C -> oresat-passives:L3216C; symbol HGS_Reflector-eagle-import:L-EUL3216C -> Device:L_Small
- PCBA1: footprint WF-NP9202 -> HGS_Reflector:WF-NP9202
- PCBA2: footprint RASP_PI_0W -> oresat-misc:RASP_PI_0W
- U1, U5: footprint Package_TO_SOT_SMD:SOT-23-5 -> oresat-ics:SOT-23 LP2985
- U2, U7: footprint SON50P200X200X95-9N-D -> oresat-ics:TQP3M9037
- U4: footprint oresat-ics:QPQ1907SR -> oresat-ics:QPQ1907
- U8: footprint Bidirectional_Amp:FIL_B39162B9417K610 -> oresat-ics:QPQ1907
Connections:
- net GND: now also J5.1 (GND@0), J5.2 (GND@1), C22.2, D1.1 (K); no longer J5.SHIELD (GND)
- net at R9.1: now also D1.2 (A)
- net at C19.2: now also J5.FEED (SIGNAL), L5.1; no longer C6.1
- net at C18.1: now also C6.1
- net at R7.1: now also D2.2 (A)
- net at C18.2: now also C22.1, L5.2; no longer J5.CENTER (SIG)
- net at J3.5: now also D2.1 (K)
Other:
- note removed: "16 turn 2.422 GHz Helical"
- note removed: "CUT+JUMPER TO ANTENNA"
- note removed: "NCS3-272+ Test Circuit"
- note removed: "NCS3-72+?"
- moved on the sheet: C1, C10, C11, C12, C13, C14, C15, C16, C18, C2, C20, C21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

Commit message: organized schematic
Other:
- moved on the sheet: C10, C20, C21, C9, D1, D2, E4, E5, J2, J3, J7, PCBA1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

Commit message: minor layout changes
Connections:
- net RF4: now reaches C14.1, L2.1, U2.7 (RF_OUT)
- net RF1: now reaches C19.2, J5.FEED (SIGNAL), L5.1
- net RF2: now reaches C18.2, C22.1, L5.2
- net RF3: now reaches C6.2, U2.2 (RF_IN)
Changed lines of the file:
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@@
+		)
+	)
+	(label "RF3"
+		(at 81.28 212.09 0)
+		(fields_autoplaced yes)
+		(effects
+			(font
+				(size 1.27 1.27)
+			)
+			(justify left bottom)
+		)
+	)
+	(label "RF4"
+		(at 121.92 212.09 0)
+		(fields_autoplaced yes)
+		(effects
+			(font
+				(size 1.27 1.27)
+			)
+			(justify left bottom)
+		)
+	)
+	(label "RF1"
+		(at 30.48 212.09 0)
+		(fields_autoplaced yes)
+		(effects
+			(font
+				(size 1.27 1.27)
+			)
+			(justify left bottom)
+		)
+	)
+	(label "RF2"
+		(at 54.61 212.09 0)
+		(fields_autoplaced yes)
+		(effects
+			(font
+				(size 1.27 1.27)
+			)
+			(justify left bottom)
 		)
 	)

Commit message: added connection from rf track to helical at entry point
Parts:
- added J4: Conn_01x01_Pin, TestPoint:TestPoint_THTPad_D1.5mm_Drill0.7mm, symbol Connector:Conn_01x01_Pin
- added R4: R_Small_US, oresat-passives:0402-C-NOSILK, symbol Device:R_Small_US
Connections:
- net RF1: now also J4.1 (Pin_1), R4.2; no longer J5.FEED (SIGNAL)
- new net: J5.FEED (SIGNAL), R4.1
Other:
- moved on the sheet: J5
Changed lines of the file:
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@@
 	)
 	(junction
-		(at 35.56 212.09)
+		(at 182.88 167.64)
 		(diameter 0)
 		(color 0 0 0 0)
 	)
 	(junction
-		(at 182.88 167.64)
+		(at 50.8 212.09)
 		(diameter 0)
 		(color 0 0 0 0)
 	)
 	(junction
-		(at 50.8 212.09)
+		(at 33.02 212.09)
 		(diameter 0)
 		(color 0 0 0 0)
@@
 	)
 	(junction
-		(at 22.86 219.71)
+		(at 17.78 219.71)
 		(diameter 0)
 		(color 0 0 0 0)
@@
 	)
 	(junction
+		(at 35.56 212.09)
+		(diameter 0)
+		(color 0 0 0 0)
+	)
+	(junction
 		(at 187.96 153.67)
 		(diameter 0)
@@
 	(wire
 		(pts
+			(xy 31.75 212.09) (xy 33.02 212.09)
+		)
+		(stroke
+			(width 0)
+			(type default)
+		)
+	)
+	(wire
+		(pts
 			(xy 161.29 212.09) (xy 165.1 212.09)
 		)
@@
 	(wire
 		(pts
-			(xy 30.48 212.09) (xy 35.56 212.09)
-		)
-		(stroke
-			(width 0)
-			(type default)
-		)
-	)
-	(wire
-		(pts
 			(xy 187.96 153.67) (xy 193.04 153.67)
 		)
@@
 	(wire
 		(pts
-			(xy 22.86 217.17) (xy 22.86 219.71)
+			(xy 17.78 217.17) (xy 17.78 219.71)
 		)
 		(stroke
@@
 	(wire
 		(pts
-			(xy 22.86 219.71) (xy 22.86 222.25)
+			(xy 17.78 219.71) (xy 17.78 222.25)
 		)
 		(stroke
@@
 	(wire
 		(pts
+			(xy 25.4 212.09) (xy 26.67 212.09)
+		)
+		(stroke
+			(width 0)
+			(type default)
+		)
+	)
+	(wire
+		(pts
 			(xy 90.17 33.02) (xy 97.79 33.02)
 		)
@@
 	(wire
 		(pts
+			(xy 33.02 212.09) (xy 35.56 212.09)
+		)
+		(stroke
+			(width 0)
+			(type default)
+		)
+	)
+	(wire
+		(pts
 			(xy 209.55 166.37) (xy 209.55 171.45)
 		)
@@
 	)
 	(label "RF1"
-		(at 30.48 212.09 0)
+		(at 35.56 212.09 0)
 		(fields_autoplaced yes)
 		(effects
@@
 	(symbol
 		(lib_id "power:GND")
-		(at 22.86 222.25 0)
+		(at 17.78 222.25 0)
 		(unit 1)
 		(exclude_from_sim no)
@@
 		(dnp no)
 		(property "Reference" "#GND010"
-			(at 22.86 222.25 0)
+			(at 17.78 222.25 0)
 			(effects
 				(font
@@
 		)
 		(property "Value" "GND"
-			(at 20.32 224.79 0)
+			(at 15.24 224.79 0)
 			(effects
 				(font
@@
 		)
 		(property "Footprint" ""
-			(at 22.86 222.25 0)
+			(at 17.78 222.25 0)
 			(effects
 				(font
@@
 		)
 		(property "Datasheet" ""
-			(at 22.86 222.25 0)
+			(at 17.78 222.25 0)
 			(effects
 				(font
@@
 		)
 		(property "Description" "Power symbol creates a global label with name \"GND\" , ground"
-			(at 22.86 222.25 0)
+			(at 17.78 222.25 0)
 			(effects
 				(font
@@
 	)
 	(symbol
+		(lib_id "Device:R_Small_US")
+		(at 29.21 212.09 90)
+		(unit 1)
+		(exclude_from_sim no)
+		(in_bom no)
+		(on_board yes)
+		(dnp no)
+		(property "Reference" "R4"
+			(at 26.67 213.106 90)
+			(effects
+				(font
+					(size 1.27 1.27)
+				)
+			)
+		)
+		(property "Value" "R_Small_US"
+			(at 28.448 214.63 90)
+			(effects
+				(font
+					(size 1.27 1.27)
+				)
+			)
+		)
+		(property "Footprint" "oresat-passives:0402-C-NOSILK"
+			(at 29.21 212.09 0)
+			(effects
+				(font
+					(size 1.27 1.27)
+				)
+				(hide yes)
+			)
+		)
+		(property "Datasheet" "~"
+			(at 29.21 212.09 0)
+			(effects
+				(font
+					(size 1.27 1.27)
+				)
+				(hide yes)
+			)
+		)
+		(property "Description" "Resistor, small US symbol"
+			(at 29.21 212.09 0)
+			(effects
+				(font
+					(size 1.27 1.27)
+				)
+				(hide yes)
+			)
+		)
+		(pin "2"
+		)
+		(pin "1"
+		)
+		(instances
+			(project ""
+				(path "/6e315cc8-f4ea-4ab4-9729-187271e6eeaf"
+					(reference "R4")
+					(unit 1)
+				)
+			)
+		)
+	)
+	(symbol
 		(lib_id "power:GND")
 		(at 50.8 224.79 0)
@@
 	)
 	(symbol
+		(lib_id "Connector:Conn_01x01_Pin")
+		(at 33.02 207.01 270)
+		(unit 1)
+		(exclude_from_sim no)
+		(in_bom yes)
+		(on_board yes)
+		(dnp no)
+		(property "Reference" "J4"
+			(at 35.814 206.756 90)
+			(effects
+				(font
+					(size 1.27 1.27)
+				)
+			)
+		)
+		(property "Value" "Conn_01x01_Pin"
+			(at 33.528 204.47 90)
+			(effects
+				(font
+					(size 1.27 1.27)
+				)
+			)
+		)
+		(property "Footprint" "TestPoint:TestPoint_THTPad_D1.5mm_Drill0.7mm"
+			(at 33.02 207.01 0)
+			(effects
+				(font
+					(size 1.27 1.27)
+				)
+				(hide yes)
+			)
+		)
+		(property "Datasheet" "~"
+			(at 33.02 207.01 0)
+			(effects
+				(font
+					(size 1.27 1.27)
+				)
+				(hide yes)
+			)
+		)
+		(property "Description" "Generic connector, single row, 01x01, script generated"
+			(at 33.02 207.01 0)
+			(effects
+				(font
+					(size 1.27 1.27)
+				)
+				(hide yes)
+			)
+		)
+		(pin "1"
+		)
+		(instances
+			(project ""
+				(path "/6e315cc8-f4ea-4ab4-9729-187271e6eeaf"
+					(reference "J4")
+					(unit 1)
+				)
+			)
+		)
+	)
+	(symbol
 		(lib_id "power:GND")
 		(at 102.87 231.14 0)
@@
 	(symbol
 		(lib_id "oresat-connectors:U.FL")
-		(at 25.4 212.09 0)
+		(at 20.32 212.09 0)
 		(unit 1)
 		(exclude_from_sim no)
@@
 		(dnp no)
 		(property "Reference" "J5"
-			(at 15.24 208.28 0)
+			(at 10.16 208.28 0)
 			(effects
 				(font
@@
 		)
 		(property "Value" "132134-10"
-			(at 15.24 209.55 0)
+			(at 10.16 209.55 0)
 			(effects
 				(font
@@
 		)
 		(property "Footprint" "oresat-connectors:U.FL"
-			(at 24.13 208.788 0)
+			(at 19.05 208.788 0)
 			(effects
 				(font
@@
 		)
 		(property "Datasheet" "~"
-			(at 25.4 212.09 0)
+			(at 20.32 212.09 0)
 			(effects
 				(font
@@
 		)
 		(property "Description" "coaxial connector (BNC, SMA, SMB, SMC, Cinch/RCA, LEMO, ...)"
-			(at 25.4 212.09 0)
+			(at 20.32 212.09 0)
 			(effects
 				(font
